Commit message: t

File: assets/Assem1/urdf/Assem1.urdf (robot description, URDF)
Before this commit: robot Assem1, 6 links, 5 joints
Joints:
- joint joint1: limit lower=1.5 upper=1.5 effort=0 velocity=1 -> lower=-1.5 upper=1.5 effort=0 velocity=1
- joint joint2: limit lower=1.5 upper=1.5 effort=0 velocity=1 -> lower=-1.5 upper=1.5 effort=0 velocity=1
- joint joint3: limit lower=1.5 upper=1.5 effort=0 velocity=1 -> lower=-1.5 upper=1.5 effort=0 velocity=1
- joint joint4: limit lower=1.5 upper=1.5 effort=0 velocity=1 -> lower=-1.5 upper=1.5 effort=0 velocity=1
- joint joint5: limit lower=1.5 upper=1.5 effort=0 velocity=1 -> lower=-1.5 upper=1.5 effort=0 velocity=1

File: assets/button/urdf/simple_button.urdf (robot description, URDF)
Before this commit: robot simple_push_button, 3 links, 2 joints
Links:
- link simple_push_button__base: geometry collision mesh filename=meshes/base_button.dae scale=0.1 0.1 0.1; visual mesh filename=meshes/base_button.dae scale=0.1 0.1 0.1
- link simple_push_button__button: geometry collision mesh filename=meshes/button.dae scale=0.1 0.1 0.1; visual mesh filename=meshes/button.dae scale=0.1 0.1 0.1
- link simple_push_button__cylinder: geometry collision mesh filename=meshes/base_cylinder.dae scale=0.1 0.1 0.1; visual mesh filename=meshes/base_cylinder.dae scale=0.1 0.1 0.1
